File: uniphob_main/uniphob_main.kicad_pcb (KiCad board)
At the start: 2 copper layers, 76 parts, among them J3 Conn_01x02_Pin, P1 Endpoint, Q1 BSS138, Q2 BSS138, Q3 BSS138, Q4 Q_NMOS_GSD, Q5 Q_PMOS_GDS, Q6 Q_NMOS_GSD, U10 RP2040, U11 LP3986-33B3F, U9 W25Q128JVS, Y1 Crystal_GND3

Commit message: Checkpoint
Parts:
- added C20: 100n, Capacitor_SMD:C_0402_1005Metric, F.Cu at (97.1, 39.2)
- added C21: 100n, Capacitor_SMD:C_0402_1005Metric, F.Cu at (147.1, 39.4)
- added D5: BAS16VY,115, uniphob_footprints:SOT-363_SC-70-6, F.Cu at (119.1, 43.7)
- added D6: BAS16VY,115, uniphob_footprints:SOT-363_SC-70-6, F.Cu at (122.2, 43.7)
- added D7: BAS16VY,115, uniphob_footprints:SOT-363_SC-70-6, F.Cu at (125.2, 43.7)
- added D8: BAS16VY,115, uniphob_footprints:SOT-363_SC-70-6, F.Cu at (128.3, 43.7)
- added J1: USB_C_Receptacle, uniphob_footprints:Shou Han Type-C 24P QCHT, F.Cu at (68.1, 81.7)
- added J2: Conn_01x06_Female, uniphob_footprints:GCC_Header_Straight_1x06_Pitch2.00mm, B.Cu at (114.8, 31.5)
- added J4: Rumble, uniphob_footprints:rumble_pins, B.Cu at (103.0, 69.4)
- added J5: Conn_02x04_Counter_Clockwise, Connector_PinSocket_2.00mm:PinSocket_2x04_P2.00mm_Vertical, B.Cu at (108.5, 27.6)
- added J6: Conn_01x02_Socket, Connector_PinSocket_2.00mm:PinSocket_1x02_P2.00mm_Vertical, F.Cu at (183.8, 60.1)
- added J7: Conn_01x05_Pin, uniphob_footprints:molex_5034800540, B.Cu at (179.3, 76.5)
- added J8: Conn_01x02_Socket, Connector_PinSocket_2.00mm:PinSocket_1x02_P2.00mm_Vertical, F.Cu at (63.8, 60.2)
- added L1: SK6805-EC-15, uniphob_footprints:SK6805-EC-15, F.Cu at (162.3, 56.9)
- added L3: SK6805-EC-15, uniphob_footprints:SK6805-EC-15, F.Cu at (150.3, 54.8)
- added L5: SK6805-EC-15, uniphob_footprints:SK6805-EC-15, F.Cu at (177.7, 53.6)
- added L7: SK6805-EC-15, uniphob_footprints:SK6805-EC-15, F.Cu at (161.4, 42.6)
- added RV1: Slider_GCC-Gamecube_MB, uniphob_footprints:GCC_Slider, B.Cu at (99.0, 37.2)
- added RV2: Slider_GCC-Gamecube_MB, uniphob_footprints:GCC_Slider, B.Cu at (149.0, 37.2)
- added SW1: GL18_SW, uniphob_footprints:GL18, F.Cu at (82.8, 52.2)
- added SW10: DPAD, uniphob_footprints:Dpad_Contact_TL3315NF_2_gba, F.Cu at (93.9, 82.2)
- added SW11: DPAD, uniphob_footprints:Dpad_Contact_TL3315NF_2_gba, F.Cu at (109.6, 82.2)
- added SW12: BPAD, uniphob_footprints:Z_Switch_Edge_Omron, F.Cu at (73.9, 36.6)
- added SW14: BPAD, uniphob_footprints:Z_Switch_Edge_Omron, F.Cu at (174.2, 36.6)
- added SW16: BPAD, uniphob_footprints:Start_Contact, F.Cu at (124.0, 52.2)
- added SW2: GL18_SW, uniphob_footprints:GL18, F.Cu at (-43.7, 43.4)
- added SW3: TS-1187A-B-A-B, uniphob_footprints:SW_TS-1187A-B-A-B, F.Cu at (-14.3, 8.62)
- added SW4: BPAD, uniphob_footprints:ABXY_Contact_Omron_Switch_Circley, F.Cu at (165.2, 52.3)
- added SW5: BPAD, uniphob_footprints:ABXY_Contact_Omron_Switch_Circley, F.Cu at (150.0, 59.8)
- added SW6: BPAD, uniphob_footprints:ABXY_Contact_Omron_Switch_Circley, F.Cu at (179.7, 48.8)
- added SW7: BPAD, uniphob_footprints:ABXY_Contact_Omron_Switch_Circley, F.Cu at (161.4, 37.9)
- added SW8: DPAD, uniphob_footprints:Dpad_Contact_TL3315NF_2_gba, F.Cu at (101.8, 74.3)
- added SW9: DPAD, uniphob_footprints:Dpad_Contact_TL3315NF_2_gba, F.Cu at (101.8, 90.0)
- added U1: ST_LSM6, uniphob_footprints:LGA14, F.Cu at (102.1, 54.4)
- added U2: ST_LSM6, uniphob_footprints:LGA14, F.Cu at (171.8, 70.5)
- added U3, U4: GH39F (Hall SOT23), uniphob_footprints:GH39F, F.Cu at (82.8, 52.2)
- added U5: GH39F (Hall SOT23), uniphob_footprints:GH39F, F.Cu at (-24.4, 30.0)
- added U6: GH39F (Hall SOT23), uniphob_footprints:GH39F, F.Cu at (-24.4, 33.9)
- added U7: MCP3002, uniphob_footprints:SOIC-8_3.9x4.9mm_P1.27mm, F.Cu at (101.1, 43.2)
- added U8: MCP3002, uniphob_footprints:SOIC-8_3.9x4.9mm_P1.27mm, F.Cu at (179.3, 70.4)
- moved C3 145.8 mm to (171.8, 73.2), turned to 180 degrees
- moved C4 141.6 mm to (169.2, 70.5), turned to 90 degrees
- moved R5 138.4 mm to (161.8, 67.0), turned to -90 degrees
- moved U10 120.6 mm to (138.5, 45.5)
- moved R3 113.5 mm to (137.9, 30.7), turned to 90 degrees
- moved R4 112.8 mm to (137.5, 51.3), turned to 180 degrees
- moved C17 109.7 mm to (124.8, 27.0), turned to 90 degrees
- moved R13 109.7 mm to (140.3, 39.7), turned to -90 degrees
- moved R11 109.6 mm to (140.0, 50.8), turned to 90 degrees
- moved R10 108.8 mm to (136.2, 38.7)
- moved R12 108.6 mm to (139.2, 39.7), turned to -90 degrees
- moved C12 105.5 mm to (143.3, 39.7), turned to 90 degrees
- moved C11 104.6 mm to (139.0, 50.8), turned to -90 degrees
- moved C10 104.3 mm to (141.3, 39.7), turned to -90 degrees
- moved C13 104.2 mm to (142.3, 39.7), turned to 90 degrees
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Routing:
- net SPI_RX: track 0.00 -> 136.6 mm, vias 0 -> 9
- net SPI_TX: track 0.00 -> 130.9 mm, vias 0 -> 7
- net SPI_CK: track 0.00 -> 124.2 mm, vias 0 -> 8
- net L_Pull: track 0.00 -> 95.5 mm, vias 0 -> 4
- net DD_Pull: track 0.00 -> 74.8 mm, vias 0 -> 7
- net RS_BUTTON: track 0.00 -> 72.5 mm, vias 0 -> 5
- net DL_Pull: track 0.00 -> 70.4 mm, vias 0 -> 3
- net RADC_CS: track 0.00 -> 65.8 mm, vias 0 -> 4
- net DR_Pull: track 0.00 -> 65.4 mm, vias 0 -> 3
- net L_ANALOG: track 0.00 -> 63.0 mm, vias 0 -> 2
- net IMU1_CS: track 0.00 -> 61.9 mm, vias 0 -> 8
- net IMU0_CS: track 0.00 -> 53.8 mm, vias 0 -> 4
- net DU_Pull: track 0.00 -> 53.0 mm, vias 0 -> 3
- net ZL_Pull: track 0.00 -> 50.7 mm, vias 0 -> 2
- net LADC_CS: track 0.00 -> 46.5 mm, vias 0 -> 4
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Other:
- board outline added: 125.5 x 72.9 mm
- copper layers 2 -> 4

Commit message: ROUTING
Parts:
- removed C7, C8: .047u, Capacitor_SMD:C_0603_1608Metric_Pad1.08x0.95mm_HandSolder
- removed R8, R9: 1k, Resistor_SMD:R_0402_1005Metric
- removed SW2: GL18_SW, uniphob_footprints:GL18
- removed TP10, TP11, TP12, TP13, TP14, TP15, TP16, TP6, TP8, TP9: TestPoint, TestPoint:TestPoint_Pad_D1.5mm
- removed U5, U6: GH39F (Hall SOT23), uniphob_footprints:GH39F
- added R25: 5.1k, Resistor_SMD:R_0603_1608Metric_Pad0.98x0.95mm_HandSolder, F.Cu at (120.0, 36.9)
- added R26: 5.1k, Resistor_SMD:R_0603_1608Metric_Pad0.98x0.95mm_HandSolder, F.Cu at (121.6, 36.9)
- added REF**: LOGO, uniphob_footprints:Ghost Logo Small, F.Cu at (76.2, 68.3)
- added REF**: HHL_Logo, uniphob_footprints:HHL_Logo, F.Cu at (66.0, 70.6)
- J1: value USB_C_Receptacle -> USB4105-GF-A-060; footprint uniphob_footprints:Shou Han Type-C 24P QCHT -> uniphob_footprints:GCT_USB4105-GF-A-060
- J5: footprint Connector_PinSocket_2.00mm:PinSocket_2x04_P2.00mm_Vertical -> uniphob_footprints:PinSocket_2x05_P2.00mm_Vertical
- moved SW3 159.3 mm to (143.2, 32.6), turned to -90 degrees
- moved TP5 89.6 mm to (102.6, 67.5)
- moved TP7 69.2 mm to (81.4, 70.0)
- moved TP1 67.7 mm to (69.3, 66.6)
- moved TP2 67.6 mm to (72.4, 67.2)
- moved J2 6.89 mm to (118.8, 25.9)
- moved F2 5.99 mm to (125.0, 28.9)
- moved F1 5.82 mm to (124.9, 26.6), turned to 0 degrees
- moved D2 4.95 mm to (132.8, 30.5)
- moved R1 4.84 mm to (62.9, 75.5)
- moved C17 3.84 mm to (128.6, 27.7)
- moved D1 3.79 mm to (131.7, 28.3)
- moved C19 3.79 mm to (132.2, 26.5)
- moved J5 3.37 mm to (108.8, 31.0)
- moved C18 3.02 mm to (129.3, 31.4), turned to 0 degrees
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Connections:
- net /CC1 renamed Net-(J1-CC1)
- net /CC2 renamed Net-(J1-CC2)
- J5 pad 5: +5V_PRE -> CC1
- J5 pad 6: +3.3V_PRE -> CC2
- J5 pad 7: D- -> +5V_PRE
- J5 pad 8: D+ -> +3.3V_PRE
Routing:
- net Scan_C: track 27.8 -> 199.9 mm, vias 0 -> 5
- net D-: track 33.2 -> 129.4 mm, vias 1 -> 4
- net +5V_PRE: track 12.7 -> 106.8 mm, vias 1 -> 3
- net D+: track 33.3 -> 121.6 mm, vias 1 -> 4
- net R_Pull: track 1.19 -> 85.8 mm, vias 1 -> 6
- net Scan_B: track 35.0 -> 110.7 mm, vias 0 -> 6
- net Scan_A: track 0.00 -> 74.8 mm, vias 0 -> 5
- net LS_BUTTON: track 3.50 -> 73.7 mm
- net R_BRAKE: track 1.68 -> 66.4 mm, vias 0 -> 2
- net X_Pull: track 16.9 -> 79.3 mm, vias 1 -> 3
- net +5V: track 10.8 -> 67.2 mm, vias 1 -> 3
- net RUMBLE: track 1.03 -> 56.4 mm, vias 0 -> 3
- net ZR_Pull: track 1.78 -> 55.0 mm, vias 1 -> 2
- net +3V3: track 34.1 -> 86.2 mm, vias 1 -> 26
- net Y_Pull: track 14.1 -> 61.6 mm, vias 1 -> 4
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- added copper zone on In2.Cu, net +3V3
- added copper zone on B.Cu, net GND
- added copper zone on F.Cu, net GND
- added copper zone on In1.Cu, net GND
Other:
- board text added: "GND->"
- board text added: "UniPhob V1 Design by Mitch & Phob Dev Team"

Commit message: Routing done
Parts:
- added J9: Conn_01x05_Pin, Connector_PinHeader_2.00mm:PinHeader_1x05_P2.00mm_Vertical, F.Cu at (184.3, 80.3)
- moved R26 18.2 mm to (104.1, 31.8)
- moved R25 15.3 mm to (105.7, 31.8)
- moved J5 8.23 mm to (116.8, 29.1), turned to 90 degrees
- moved TP5 1.30 mm to (101.9, 66.4)
Routing:
- net RX: track 5.15 -> 12.8 mm
- net RY: track 5.70 -> 13.3 mm
- net D+: track 121.6 -> 128.8 mm
- net RS_BUTTON: track 73.2 -> 78.8 mm
- net N_LATCH: track 11.4 -> 6.70 mm, vias 2 -> 0
- net CC2: track 10.5 -> 5.90 mm
- net +5V_PRE: track 106.8 -> 111.0 mm
- net CC1: track 6.85 -> 3.28 mm
- net GND: track 37.6 -> 34.7 mm, vias 22 -> 21
- net N_CLOCK: track 6.34 -> 8.61 mm, vias 0 -> 2
- net D-: track 129.4 -> 131.7 mm, vias 4 -> 3
- net +5V: track 67.2 -> 68.6 mm
Other:
- outline, holes or cut-outs redrawn
- board text added: "3.3v X Y Btn GND"
